Commit message: configuration changes

File: svenzva_description/robots/svenzva_arm.urdf (robot description, URDF)
Before this commit: robot svenzva_arm, 9 links, 8 joints
Joints:
- joint joint_2: origin xyz=-0.00700000000002309 0.0549537554950766 0 rpy=1.66359981346176E-15 -1.0547118733939E-15 -1.68424757676597 -> xyz=-0.00700000000002309 0.0549537554950766 0 rpy=0 0 -1.88424757676597
- joint joint_4: origin xyz=0.00094769 0.228 0 rpy=2.5315 -1.5708 0 -> xyz=0.00094769 0.228 0 rpy=0 -1.5708 0
- joint joint_5: origin xyz=-0.002 0.1909 0 rpy=1.0193 1.5708 0 -> xyz=-0.002 0.1909 0 rpy=0 0 0
- joint joint_6: origin xyz=-0.00025 0 0.0763 rpy=1.5708 -1.7764E-15 1.5478 -> xyz=-0.00025 0 0.0763 rpy=1.5708 0 1.5478
- joint link_3: origin xyz=-0.07037 0.21525 0 rpy=2.3606 -1.5708 0 -> xyz=-0.07037 0.21525 0 rpy=0.3 -1.5708 0

Commit message: changes to urdf for latest design, and major changes to driver position intialization to match actual robot state correctly.

File: svenzva_description/robots/svenzva_arm.urdf (robot description, URDF)
Before this commit: robot svenzva_arm, 9 links, 8 joints
Links:
- removed link link7
- removed link link8
- added link link_finger_1, mass 0.0100194667897186; collision mesh filename=package://svenzva_description/meshes/link_finger_1.STL; visual mesh filename=package://svenzva_description/meshes/link_finger_1.STL
- added link link_finger_2, mass 0.0100194667897082; collision mesh filename=package://svenzva_description/meshes/link_finger_2.STL; visual mesh filename=package://svenzva_description/meshes/link_finger_2.STL
- link base_link: mass 0.0440503098818098 -> 0.0440503113116943
- link link_1: mass 0.0905550798572669 -> 0.0925085972682552
- link link_2: mass 0.0990854582025164 -> 0.111498195078862
- link link_3: mass 0.0987656165583022 -> 0.095277105355898
- link link_4: mass 0.0667180708029316 -> 0.0630903380817815
- link link_5: mass 0.0487770287268765 -> 0.0564481780820506
- link link_6: mass 0.00316138019909441 -> 0.0901281281958769
Joints:
- removed joint joint7
- removed joint joint8
- removed joint link_3
- added joint finger_1: type fixed, parent link_6, child link_finger_1, origin xyz=0.0222737654014398 0.0365533597460683 0.0727446167971825 rpy=-1.5707963267949 1.33127052458092 1.55441469771021, axis 0 0 0
- added joint finger_2: type fixed, parent link_6, child link_finger_2, origin xyz=-0.0225240000000001 -0.0368716233284919 0.0727685295284096 rpy=-1.57079632679489 1.32996070258273 -1.58717795587957, axis 0 0 0
- added joint joint_3: type continuous, parent link_2, child link_3, origin xyz=0.226700000000002 -0.0266129086637006 0 rpy=3.14159265358979 0.0162072294682094 -1.40791300798038E-15, axis 0 1 0
- joint joint_1: axis 0 -1 0 -> 0 1 0; origin xyz=0 0 0 rpy=1.57079 0.0 0.0 -> xyz=0.183061688655131 -0.012 0.036500000000004 rpy=1.5707963267949 -6.12285515858645E-17 -1.5632010942264
- joint joint_2: axis 0 0 -1 -> 0 -1 0; origin xyz=-0.00700000000002309 0.0549537554950766 0 rpy=0 0 -1.88424757676597 -> xyz=-0.007 0.057 0 rpy=1.5708 -1.3131E-15 1.5993
- joint joint_4: axis 1 0 0 -> 0 1 0; origin xyz=0.00094769 0.228 0 rpy=0 -1.5708 0 -> xyz=0.137700000000002 -0.0270129086636999 0 rpy=-1.5707963267949 -9.0205620750794E-16 -0.000965169435000781
- joint joint_5: axis -1 0 0 -> 0 -1 0; origin xyz=-0.002 0.1909 0 rpy=0 0 0 -> xyz=0.1282 0.00249999999999978 0 rpy=-1.5707963267949 4.61393076522931E-15 3.13849286930343
- joint joint_6: axis 0 1 0 -> 0 0 1; origin xyz=-0.00025 0 0.0763 rpy=1.5708 0 1.5478 -> xyz=-0.0838128178357174 -0.00757500000000258 -0.00400000000009831 rpy=1.57079632678785 -1.56490357222949 -1.57079632678785

Commit message: modified urdf such that the end effector is included in moveit demo

File: svenzva_description/robots/svenzva_arm.urdf (robot description, URDF)
Before this commit: robot svenzva_arm, 9 links, 8 joints
Links:
- removed link link_finger_1
- removed link link_finger_2
- link link_6: mass 0.0901281281958769 -> 0.110167061775322
Joints:
- removed joint finger_1
- removed joint finger_2
- joint joint_1: origin xyz=0.183061688655131 -0.012 0.036500000000004 rpy=1.5707963267949 -6.12285515858645E-17 -1.5632010942264 -> xyz=0.18306 -0.012 0.0365 rpy=1.5708 -6.1229E-17 -1.5632
- joint joint_2: limit (none) -> lower=-2.0 upper=2.0 effort=30 velocity=3.0; type continuous -> revolute
- joint joint_3: limit (none) -> lower=-2.0 upper=2.0 effort=30 velocity=3.0; origin xyz=0.226700000000002 -0.0266129086637006 0 rpy=3.14159265358979 0.0162072294682094 -1.40791300798038E-15 -> xyz=0.2267 -0.026613 0 rpy=3.1416 0.016207 -1.4079E-15; type continuous -> revolute
- joint joint_4: limit (none) -> lower=-2.0 upper=2.0 effort=30 velocity=3.0; origin xyz=0.137700000000002 -0.0270129086636999 0 rpy=-1.5707963267949 -9.0205620750794E-16 -0.000965169435000781 -> xyz=0.1377 -0.027013 0 rpy=-1.5708 -9.0206E-16 -0.00096517; type continuous -> revolute
- joint joint_5: limit (none) -> lower=-1.55 upper=1.65 effort=30 velocity=3.0; origin xyz=0.1282 0.00249999999999978 0 rpy=-1.5707963267949 4.61393076522931E-15 3.13849286930343 -> xyz=0.1282 0.0025 0 rpy=-1.5708 4.6139E-15 3.1385; type continuous -> revolute
- joint joint_6: origin xyz=-0.0838128178357174 -0.00757500000000258 -0.00400000000009831 rpy=1.57079632678785 -1.56490357222949 -1.57079632678785 -> xyz=-0.083813 -0.007575 -0.004 rpy=1.5708 -1.5649 -1.5708

Commit message: updated urdf model and meshes. updated driver init values to be more accurate. moveit updated with EF link

File: svenzva_description/robots/svenzva_arm.urdf (robot description, URDF)
Before this commit: robot svenzva_arm, 7 links, 6 joints
Links:
- added link ee_link
- link link_1: mass 0.0925085972682552 -> 0.092508596891218
- link link_2: mass 0.111498195078862 -> 0.111498195075492
- link link_3: mass 0.095277105355898 -> 0.0953320551486545
- link link_4: mass 0.0630903380817815 -> 0.0669634671076673
- link link_5: mass 0.0564481780820506 -> 0.061656
- link link_6: mass 0.110167061775322 -> 0.1101
Joints:
- added joint ee_joint: type fixed, parent link_6, child ee_link, origin xyz=0.015 0 0.15
- joint joint_1: origin xyz=0.18306 -0.012 0.0365 rpy=1.5708 -6.1229E-17 -1.5632 -> xyz=0.183061688655131 -0.0119999999999999 0.0385000000000039 rpy=-1.5707963267949 -6.12303176911189E-17 -1.5707963267949
- joint joint_2: origin xyz=-0.007 0.057 0 rpy=1.5708 -1.3131E-15 1.5993 -> xyz=-0.00699999999999987 -0.055 0 rpy=1.57079632679488 -1.38777878078116E-15 -1.57079632679488
- joint joint_3: axis 0 1 0 -> 0 -1 0; origin xyz=0.2267 -0.026613 0 rpy=3.1416 0.016207 -1.4079E-15 -> xyz=0.2267 0 0 rpy=1.72604985859693E-14 -1.72604985859694E-14 -1.38777878078145E-15
- joint joint_4: axis 0 1 0 -> 0 -1 0; origin xyz=0.1377 -0.027013 0 rpy=-1.5708 -9.0206E-16 -0.00096517 -> xyz=0.1377 -0.000399999966000264 0 rpy=-1.5707963267949 -5.02171683388957E-18 -0.00827101619955667
- joint joint_5: origin xyz=0.1282 0.0025 0 rpy=-1.5708 4.6139E-15 3.1385 -> xyz=0.1282 -0.00269999999999876 0 rpy=-1.5707963267949 -2.77729228503887E-15 -3.14159265358979
- joint joint_6: axis 0 0 1 -> 0 0 -1; origin xyz=-0.083813 -0.007575 -0.004 rpy=1.5708 -1.5649 -1.5708 -> xyz=-0.0891078454541699 -0.000699989976996301 -0.0124999999999946 rpy=-1.5707963267949 -1.47451495458029E-15 1.5707963267949

Commit message: modified urdf for correct movement about axis

File: svenzva_description/robots/svenzva_arm.urdf (robot description, URDF)
Before this commit: robot svenzva_arm, 8 links, 7 joints
Joints:
- joint joint_1: axis 0 1 0 -> 0 -1 0
- joint joint_6: axis 0 0 -1 -> 0 0 1

Commit message: lots of changes.

File: svenzva_description/robots/svenzva_arm.urdf (robot description, URDF)
Before this commit: robot svenzva_arm, 8 links, 7 joints
Joints:
- joint joint_2: limit lower=-2.0 upper=2.0 effort=30 velocity=3.0 -> lower=-2.0 upper=2.0 effort=30 velocity=1.0
- joint joint_3: limit lower=-2.0 upper=2.0 effort=30 velocity=3.0 -> lower=-2.3 upper=2.3 effort=30 velocity=1.0
- joint joint_4: limit lower=-2.0 upper=2.0 effort=30 velocity=3.0 -> lower=-2.15 upper=2.15 effort=30 velocity=1.0
- joint joint_5: limit lower=-1.55 upper=1.65 effort=30 velocity=3.0 -> lower=-1.85 upper=1.85 effort=30 velocity=1.0

Commit message: changes in urdf for better precision, hacky additions to an alternate controller to set driver configs

File: svenzva_description/robots/svenzva_arm.urdf (robot description, URDF)
Before this commit: robot svenzva_arm, 8 links, 7 joints
Joints:
- joint joint_1: limit (none) -> lower=-3.14 upper=3.14 effort=30 velocity=1.0; type continuous -> revolute
- joint joint_6: limit (none) -> lower=-3.14 upper=3.14 effort=30 velocity=1.0; type continuous -> revolute

Commit message: fixed wrist joint limits bug

File: svenzva_description/robots/svenzva_arm.urdf (robot description, URDF)
Before this commit: robot svenzva_arm, 8 links, 7 joints
Joints:
- joint joint_6: limit lower=-3.14 upper=3.14 effort=30 velocity=1.0 -> lower=-6.0 upper=0.0 effort=30 velocity=1.0

Commit message: added new urdf for geared design with joint limits

File: svenzva_description/robots/svenzva_arm.urdf (robot description, URDF)
Before this commit: robot svenzva_arm, 8 links, 7 joints
Links:
- removed link ee_link
- link base_link: mass 0.0440503113116943 -> 0.0723639514810396
- link link_1: mass 0.092508596891218 -> 0.176002844262561
- link link_2: mass 0.111498195075492 -> 0.375844350415876
- link link_3: mass 0.0953320551486545 -> 0.31163055657814
- link link_4: mass 0.0669634671076673 -> 0.227468523944598
- link link_5: mass 0.061656 -> 0.151584942075443
- link link_6: mass 0.1101 -> 0.322937867529949
Joints:
- removed joint ee_joint
- joint joint_1: axis 0 -1 0 -> 0 1 0; origin xyz=0.183061688655131 -0.0119999999999999 0.0385000000000039 rpy=-1.5707963267949 -6.12303176911189E-17 -1.5707963267949 -> xyz=0.013 0 0.040487 rpy=1.5708 -1.1432E-16 -0.01434
- joint joint_2: axis 0 -1 0 -> 0 0 -1; origin xyz=-0.00699999999999987 -0.055 0 rpy=1.57079632679488 -1.38777878078116E-15 -1.57079632679488 -> xyz=0 0.096463 -0.02335 rpy=4.0919E-18 -1.3762E-14 1.6E-18
- joint joint_3: axis 0 -1 0 -> 0 0 -1; limit lower=-2.3 upper=2.3 effort=30 velocity=1.0 -> lower=-2.0 upper=2.0 effort=30 velocity=1.0; origin xyz=0.2267 0 0 rpy=1.72604985859693E-14 -1.72604985859694E-14 -1.38777878078145E-15 -> xyz=0 0.2267 0.015875 rpy=6.193E-16 3.5562E-16 1.9901
- joint joint_4: axis 0 -1 0 -> 0 0 -1; limit lower=-2.15 upper=2.15 effort=30 velocity=1.0 -> lower=-2.4 upper=2.4 effort=30 velocity=1.0; origin xyz=0.1377 -0.000399999966000264 0 rpy=-1.5707963267949 -5.02171683388957E-18 -0.00827101619955667 -> xyz=0.112887803122276 -0.0849668013782555 0.0137499694500327 rpy=1.57079632679489 -1.08279352070304 2.72231120032224
- joint joint_5: axis 0 -1 0 -> 0 0 1; limit lower=-1.85 upper=1.85 effort=30 velocity=1.0 -> lower=-1.9 upper=1.9 effort=30 velocity=1.0; origin xyz=0.1282 -0.00269999999999876 0 rpy=-1.5707963267949 -2.77729228503887E-15 -3.14159265358979 -> xyz=-0.0309980883229195 0.139443213449917 0.0252374943531824 rpy=1.57079632679489 0.745906426455644 2.05879913288675
- joint joint_6: axis 0 0 1 -> 0 0 -1; origin xyz=-0.0891078454541699 -0.000699989976996301 -0.0124999999999946 rpy=-1.5707963267949 -1.47451495458029E-15 1.5707963267949 -> xyz=0.0527875432993938 0.0688570078944784 -0.0317500182541626 rpy=-1.57079632679493 1.55645636523858 2.3167027532505

Commit message: reflects the gear model correctly

File: svenzva_description/robots/svenzva_arm.urdf (robot description, URDF)
Before this commit: robot svenzva_arm, 7 links, 6 joints
Links:
- link base_link: mass 0.0723639514810396 -> 0.072364
- link link_2: mass 0.375844350415876 -> 0.375844350417551
- link link_3: mass 0.31163055657814 -> 0.31163055657781
- link link_4: mass 0.227468523944598 -> 0.227468523944588
Joints:
- joint joint_2: origin xyz=0 0.096463 -0.02335 rpy=4.0919E-18 -1.3762E-14 1.6E-18 -> xyz=0 0.0964625315349195 -0.0233499999819998 rpy=4.09187004857075E-18 -1.3761561334924E-14 1.60002689098321E-18
- joint joint_3: origin xyz=0 0.2267 0.015875 rpy=6.193E-16 3.5562E-16 1.9901 -> xyz=0 0.22669999999 0.0158749999819999 rpy=6.69447407664753E-16 1.6306400674182E-16 -0.00242557244235328
- joint joint_4: axis 0 0 -1 -> 0 0 0.999999999960484; origin xyz=0.112887803122276 -0.0849668013782555 0.0137499694500327 rpy=1.57079632679489 -1.08279352070304 2.72231120032224 -> xyz=0.00912959083561864 0.137721791833396 0.0137499861543416 rpy=-2.36709870890947 1.57079630572147 -2.36079769092609
- joint joint_5: axis 0 0 1 -> 0 0 -1; origin xyz=-0.0309980883229195 0.139443213449917 0.0252374943531824 rpy=1.57079632679489 0.745906426455644 2.05879913288675 -> xyz=0.00645000003795365 0.1377 -0.00249999436214027 rpy=0 1.5707963267949 0
- joint joint_6: axis 0 0 -1 -> 0 0 1; origin xyz=0.0527875432993938 0.0688570078944784 -0.0317500182541626 rpy=-1.57079632679493 1.55645636523858 2.3167027532505 -> xyz=0.0153032852422354 0.0855005794492288 -0.0126999817460203 rpy=-1.5707963267949 -1.55645636523858 -1.09070333872558E-05

Commit message: good changes. configuration based, mostly.

File: svenzva_description/robots/svenzva_arm.urdf (robot description, URDF)
Before this commit: robot svenzva_description, 7 links, 6 joints
Links:
- added link ee_link
Joints:
- added joint ee_joint: type fixed, parent link_6, child ee_link, origin xyz=0.015 0 0.15
- joint joint_1: limit (none) -> lower=0.0 upper=6.0 effort=30 velocity=1.0; type continuous -> revolute
- joint joint_3: axis 0 0 -1 -> 0 0 1
- joint joint_4: axis 0 0 0.999999999960484 -> 0 0 -1.0
- joint joint_5: axis 0 0 -1 -> 0 0 1

Commit message: Migration from protocol 1.0 to protocol 2.0 (#1)
* general cleanup

* many changes in package structure and general driver abilities

* updated model

* removed dae

* added cartesian vel demo

* added colors, ee_link added

* updated moveit configuration for new model

* gripper interface added. arm namespaces updated

* added jacobian computation

File: svenzva_description/robots/svenzva_arm.urdf (robot description, URDF)
Before this commit: robot svenzva_description, 8 links, 7 joints
Links:
- added link link_7, mass 0.0354585256038568; collision mesh filename=package://svenzva_description/meshes/link_7.STL; visual mesh filename=package://svenzva_description/meshes/link_7.STL
- link base_link: mass 0.072364 -> 0.506214468139727
- link link_1: mass 0.176002844262561 -> 0.153541664031025
- link link_2: mass 0.375844350417551 -> 0.281175487770198
- link link_3: mass 0.31163055657781 -> 0.246165133529195
- link link_4: mass 0.227468523944588 -> 0.211922628762084
- link link_5: mass 0.151584942075443 -> 0.164460903684414
- link link_6: mass 0.322937867529949 -> 0.195112141464075
Joints:
- added joint joint_7: type fixed, parent link_6, child link_7, origin xyz=0 0 -0.0573569998840002 rpy=-3.14159265358979 0 -3.14159265358979, axis -1 0 0, limit lower=-0.05 upper=0.05 effort=5 velocity=1.0
- joint ee_joint: origin xyz=0.015 0 0.15 -> xyz=0 0 0.0; parent link_6 -> link_7
- joint joint_1: axis 0 1 0 -> 0 0 -1; limit lower=0.0 upper=6.0 effort=30 velocity=1.0 -> lower=0 upper=6.0 effort=30 velocity=1.0; origin xyz=0.013 0 0.040487 rpy=1.5708 -1.1432E-16 -0.01434 -> xyz=0 0 0.07119999984 rpy=-1.93033535706571E-16 -1.54074395550979E-32 0
- joint joint_2: origin xyz=0 0.0964625315349195 -0.0233499999819998 rpy=4.09187004857075E-18 -1.3761561334924E-14 1.60002689098321E-18 -> xyz=0.00891249579997938 0 0.09644999999 rpy=1.5707963267949 -1.93033535706571E-16 1.5707963267949
- joint joint_3: axis 0 0 1 -> 0 0 -1; origin xyz=0 0.22669999999 0.0158749999819999 rpy=6.69447407664753E-16 1.6306400674182E-16 -0.00242557244235328 -> xyz=0 0.22770179999 0.00317500840002059 rpy=-3.14159265358979 -2.14461300673676E-15 3.14159265358979
- joint joint_4: axis 0 0 -1.0 -> 0 0 1; origin xyz=0.00912959083561864 0.137721791833396 0.0137499861543416 rpy=-2.36709870890947 1.57079630572147 -2.36079769092609 -> xyz=-0.00165000009395299 0.13769999999 0.00581250408200003 rpy=0 1.5707963267949 0
- joint joint_5: axis 0 0 1 -> 0 0 -1; origin xyz=0.00645000003795365 0.1377 -0.00249999436214027 rpy=0 1.5707963267949 0 -> xyz=0.00165000009004705 0.15039999999 -0.00158749994695297 rpy=0 1.5707963267949 0
- joint joint_6: axis 0 0 1 -> 0 0 -1; limit lower=-6.0 upper=0.0 effort=30 velocity=1.0 -> lower=0.0 upper=6.0 effort=30 velocity=1.0; origin xyz=0.0153032852422354 0.0855005794492288 -0.0126999817460203 rpy=-1.5707963267949 -1.55645636523858 -1.09070333872558E-05 -> xyz=-0.0147500000020004 0.0754999999999999 0.00142499999999982 rpy=1.5707963267949 1.5707963267949 0

Commit message: Devel merge into master (#3)
* moved previous action files. actionlib-ized gripper action.

* model updated to 4_24 version

* changes to use USB, updates to gripper actions and testing with jacobian + KDL

* made compliance for full arm. generic arm services module added. dependency changes.

* manual modifications in model to match motor zero position

* initial commit for all demo files

* added basis for cartestian velocity interpreter

* added joystick interpreter for xbox 360

* ported cartesian manager to python and added it as a driver module.

* some small changes to joy. added BSD licenses

* fixed empty link references, and a few comments

* many changes getting compliance smooth, general driver organization and threading, and improvements.

* fixed actionlib code bugs

* general changes. added joint limits to cartesian controller. modified urdf to allow turns in either direction

* added gripper response

File: svenzva_description/robots/svenzva_arm.urdf (robot description, URDF)
Before this commit: robot svenzva_description, 9 links, 8 joints
Links:
- link base_link: mass 0.506214468139727 -> 0.774961748747901; geometry collision mesh filename=package://4_25_urdf6/meshes/base_link.STL; visual mesh filename=package://4_25_urdf6/meshes/base_link.STL
- link link_1: mass 0.153541664031025 -> 0.29849024; geometry collision mesh filename=package://4_25_urdf6/meshes/link_1.STL; visual mesh filename=package://4_25_urdf6/meshes/link_1.STL
- link link_2: mass 0.281175487770198 -> 0.327742070931929; geometry collision mesh filename=package://4_25_urdf6/meshes/link_2.STL; visual mesh filename=package://4_25_urdf6/meshes/link_2.STL
- link link_3: mass 0.246165133529195 -> 0.280463750144268; geometry collision mesh filename=package://4_25_urdf6/meshes/link_3.STL; visual mesh filename=package://4_25_urdf6/meshes/link_3.STL
- link link_4: mass 0.211922628762084 -> 0.246221245377158; geometry collision mesh filename=package://4_25_urdf6/meshes/link_4.STL; visual mesh filename=package://4_25_urdf6/meshes/link_4.STL
- link link_5: mass 0.164460903684414 -> 0.163854288137822; geometry collision mesh filename=package://4_25_urdf6/meshes/link_5.STL; visual mesh filename=package://4_25_urdf6/meshes/link_5.STL
- link link_6: mass 0.195112141464075 -> 0.251621037329208; geometry collision mesh filename=package://4_25_urdf6/meshes/link_6.STL; visual mesh filename=package://4_25_urdf6/meshes/link_6.STL
- link link_7: mass 0.0354585256038568 -> 0.0478690095652066; geometry collision mesh filename=package://4_25_urdf6/meshes/link_finger_1.STL; visual mesh filename=package://4_25_urdf6/meshes/link_finger_1.STL
Joints:
- joint ee_joint: parent link_7 -> link_6
- joint joint_1: limit lower=0 upper=6.0 effort=30 velocity=1.0 -> lower=-3.14 upper=3.14 effort=30 velocity=1.0; origin xyz=0 0 0.07119999984 rpy=-1.93033535706571E-16 -1.54074395550979E-32 0 -> xyz=0 0 0.06485 rpy=0 0 -1.5708
- joint joint_2: limit lower=-2.0 upper=2.0 effort=30 velocity=1.0 -> lower=-2 upper=2 effort=30 velocity=1.0; origin xyz=0.00891249579997938 0 0.09644999999 rpy=1.5707963267949 -1.93033535706571E-16 1.5707963267949 -> xyz=0 -0.015113 0.1155 rpy=1.5708 0 4.3282E-16
- joint joint_3: limit lower=-2.0 upper=2.0 effort=30 velocity=1.0 -> lower=-2 upper=2 effort=30 velocity=1.0; origin xyz=0 0.22770179999 0.00317500840002059 rpy=-3.14159265358979 -2.14461300673676E-15 3.14159265358979 -> xyz=0 0.2277 -0.009226 rpy=3.1416 -1.5345E-16 3.1416
- joint joint_4: limit lower=-2.4 upper=2.4 effort=30 velocity=1.0 -> lower=-1.7 upper=1.7 effort=30 velocity=1.0; origin xyz=-0.00165000009395299 0.13769999999 0.00581250408200003 rpy=0 1.5707963267949 0 -> xyz=-0.00165 0.1377 -0.000388 rpy=0 1.5708 0
- joint joint_5: limit lower=-1.9 upper=1.9 effort=30 velocity=1.0 -> lower=-1.7 upper=1.7 effort=30 velocity=1.0; origin xyz=0.00165000009004705 0.15039999999 -0.00158749994695297 rpy=0 1.5707963267949 0 -> xyz=0.00165 0.1504 -0.0015875 rpy=0 1.5708 0
- joint joint_6: limit lower=0.0 upper=6.0 effort=30 velocity=1.0 -> lower=0 upper=6.0 effort=30 velocity=1.0; origin xyz=-0.0147500000020004 0.0754999999999999 0.00142499999999982 rpy=1.5707963267949 1.5707963267949 0 -> xyz=-0.01475 0.08 0.001425 rpy=1.5708 3.14159 0
- joint joint_7: limit lower=-0.05 upper=0.05 effort=5 velocity=1.0 -> lower=-0.05 upper=0.05 effort=30 velocity=1.0; origin xyz=0 0 -0.0573569998840002 rpy=-3.14159265358979 0 -3.14159265358979 -> xyz=0 0 -0.052509 rpy=3.1416 3.0358E-17 3.1416; type fixed -> prismatic

Commit message: fixed package path

File: svenzva_description/robots/svenzva_arm.urdf (robot description, URDF)
Before this commit: robot revel, 9 links, 8 joints
Links:
- link base_link: geometry collision mesh filename=package://svenzva_description/meshes/base_link.STL; visual mesh filename=package://svenzva_description/meshes/base_link.STL
- link link_1: geometry collision mesh filename=package://svenzva_description/meshes/link_1.STL; visual mesh filename=package://svenzva_description/meshes/link_1.STL
- link link_2: geometry collision mesh filename=package://svenzva_description/meshes/link_2.STL; visual mesh filename=package://svenzva_description/meshes/link_2.STL
- link link_3: geometry collision mesh filename=package://svenzva_description/meshes/link_3.STL; visual mesh filename=package://svenzva_description/meshes/link_3.STL
- link link_4: geometry collision mesh filename=package://svenzva_description/meshes/link_4.STL; visual mesh filename=package://svenzva_description/meshes/link_4.STL
- link link_5: geometry collision mesh filename=package://svenzva_description/meshes/link_5.STL; visual mesh filename=package://svenzva_description/meshes/link_5.STL
- link link_6: geometry collision mesh filename=package://svenzva_description/meshes/link_6.STL; visual mesh filename=package://svenzva_description/meshes/link_6.STL
- link link_7: geometry collision mesh filename=package://svenzva_description/meshes/link_finger_1.STL; visual mesh filename=package://svenzva_description/meshes/link_finger_1.STL
Joints:
- joint joint_6: limit lower=0 upper=6.0 effort=30 velocity=1.0 -> lower=0 upper=8.0 effort=30 velocity=1.0
