Commit message: added joint limits in cartesian controller; joint limit changes in urdf; moveit parameter additions; fixed bug in driver when initializing motors to velocity mode

File: svenzva_description/robots/svenzva_arm.urdf (robot description, URDF)
Before this commit: robot revel, 9 links, 8 joints
Joints:
- joint ee_joint: origin xyz=0 0 0.0 -> xyz=0 0 -0.1 rpy=3.14159 0 0
- joint joint_3: limit lower=-2 upper=2 effort=30 velocity=1.0 -> lower=-2.2 upper=2.2 effort=30 velocity=1.0
- joint joint_4: limit lower=-1.7 upper=1.7 effort=30 velocity=1.0 -> lower=-2.0 upper=2.0 effort=30 velocity=1.0

Commit message: ros_control support (#5)
* modified joint limit for cable mgmt

* control parameter changes

* additions to make teaching mode output cartesian force

* residuals from reading parmeters from file and cmdline

* makes cartesian control a little smoother

* working demo with 1 motor on protocol v1

* many changes. got minimalist demo working on MX 2.0 motor. ros_control is wrapped around command and output topics from mx_driver and mx_controllers.

* residual from merge

* changed input to be joint states

* added raw output for testing

* now supports up to 6 joints. lacks infastructure to command all joints succinctly.

* added all joints

* added gazebo support for ros_control

* added world link for simulation

* better PID value for real robot

* furthered simulation capability by employing trajectory controller. MoveIt! now able to run with gazebo sim.

* fixes and modifications for velocity control

* code cleanup

* removed test urdf

File: svenzva_description/robots/svenzva_arm.urdf (robot description, URDF)
Before this commit: robot revel, 9 links, 8 joints
Links:
- added link world
Joints:
- added joint world_joint: type fixed, parent world, child base_link

Commit message: Update Revel Joint 4 (#6)
* modified urdf and improved cartesian controller somewhat. orientation z motion is closer to expected behavior

* changes???

* updated inertial values

* added separate prismatic fingers

* added test smoothing

* compliance modifications

* new urdf

* changed urdf and moveit config

* changed driver gear ratios

* added fingers into joint state and moveit config

File: svenzva_description/robots/svenzva_arm.urdf (robot description, URDF)
Before this commit: robot revel, 10 links, 9 joints
Links:
- removed link ee_link
- removed link link_7
- added link finger_joint_2, mass 0.0220307791071739; collision mesh filename=package://svenzva_description/meshes/finger_joint_2.STL; visual mesh filename=package://svenzva_description/meshes/finger_joint_2.STL
- added link finger_link_1, mass 0.0220307791071739; collision mesh filename=package://svenzva_description/meshes/finger_link_1.STL; visual mesh filename=package://svenzva_description/meshes/finger_link_1.STL
- link base_link: mass 0.774961748747901 -> 0.761337238502044
- link link_1: mass 0.29849024 -> 0.295038974095265
- link link_2: mass 0.327742070931929 -> 0.344381379534998
- link link_3: mass 0.280463750144268 -> 0.196650631153951
- link link_4: mass 0.246221245377158 -> 0.171727164051589
- link link_5: mass 0.163854288137822 -> 0.13919813472784
- link link_6: mass 0.251621037329208 -> 0.243320868687054
Joints:
- removed joint ee_joint
- removed joint joint_7
- added joint finger_joint_1: type prismatic, parent link_6, child finger_link_1, origin xyz=0 0 -0.052509 rpy=-3.1416 -1.8964E-18 3.1416, axis 0 1 0, limit lower=0 upper=0.05 effort=0 velocity=0
- added joint finger_joint_2: type prismatic, parent link_6, child finger_joint_2, origin xyz=0 0 -0.052509 rpy=-3.1416 -1.8964E-18 3.1416, axis 0 1 0, limit lower=-0.05 upper=0 effort=0 velocity=0
- joint joint_1: limit lower=-3.14 upper=3.14 effort=30 velocity=1.0 -> lower=-3.14 upper=3.14 effort=0 velocity=0; origin xyz=0 0 0.06485 rpy=0 0 -1.5708 -> xyz=0 0 0.0762 rpy=0 0 -4.404E-17
- joint joint_2: limit lower=-2 upper=2 effort=30 velocity=1.0 -> lower=-2 upper=2 effort=0 velocity=0; origin xyz=0 -0.015113 0.1155 rpy=1.5708 0 4.3282E-16 -> xyz=-0.007325 0 0.10542 rpy=1.5708 0 -1.5708
- joint joint_3: limit lower=-2.2 upper=2.2 effort=30 velocity=1.0 -> lower=-2 upper=2 effort=0 velocity=0; origin xyz=0 0.2277 -0.009226 rpy=3.1416 -1.5345E-16 3.1416 -> xyz=0 0.2277 0.00635 rpy=3.1416 -2.0986E-16 3.1416
- joint joint_4: limit lower=-2.0 upper=2.0 effort=30 velocity=1.0 -> lower=-5.0 upper=3.867165 effort=0 velocity=0; origin xyz=-0.00165 0.1377 -0.000388 rpy=0 1.5708 0 -> xyz=-0.020448 0.11835 0.0083512 rpy=-1.5672 1.5708 0
- joint joint_5: limit lower=-1.7 upper=1.7 effort=30 velocity=1.0 -> lower=-1.7 upper=1.7 effort=0 velocity=0; origin xyz=0.00165 0.1504 -0.0015875 rpy=0 1.5708 0 -> xyz=-0.0010724 -2.0879E-05 0.08245 rpy=1.5708 -0.0035837 -1.5708
- joint joint_6: limit lower=0 upper=8.0 effort=30 velocity=1.0 -> lower=-1.565 upper=1.565 effort=0 velocity=0; origin xyz=-0.01475 0.08 0.001425 rpy=1.5708 3.14159 0 -> xyz=-0.014463 0.080052 0.001425 rpy=1.5744 -1.5708 0

Commit message: Add Kinesthetic Teaching interface (#8)
* minimal working curses menu

* added functionality for recording arm state and gripper state.

* add playback options

* new urdf

* added fingers, transmissions

* added gripper actions, added playback functionality

* bug fixes. can save successfully save and replay gripper states

* fixes joint_state playback bugs

* made joint action async; added stall condition detection in KT console

* modified srdf for new urdf

* fixes merged issues with new urdf. updates moveit.

* class description

* changed cartesian_velocity scaling algorithm. arm movement greatly improved

* catkinized description package. removed incompatible demonstration files.

File: svenzva_description/robots/svenzva_arm.urdf (robot description, URDF)
Before this commit: robot revel, 10 links, 9 joints
Links:
- link base_link: mass 0.761337238502044 -> 0.722020764728074
- link link_2: mass 0.344381379534998 -> 0.350557648873674
- link link_3: mass 0.196650631153951 -> 0.227860881806706
- link link_4: mass 0.171727164051589 -> 0.174540765744632
- link link_5: mass 0.13919813472784 -> 0.133021865517638
- link link_6: mass 0.243320868687054 -> 0.243320868551208
Joints:
- joint finger_joint_1: axis 0 1 0 -> -1 0 0
- joint finger_joint_2: axis 0 1 0 -> -1 0 0
- joint joint_1: origin xyz=0 0 0.0762 rpy=0 0 -4.404E-17 -> xyz=0 0 0.0762 rpy=0 0 0
- joint joint_3: origin xyz=0 0.2277 0.00635 rpy=3.1416 -2.0986E-16 3.1416 -> xyz=0 0.2277 0.00635 rpy=3.1416 0 3.1416
- joint joint_4: limit lower=-5.0 upper=3.867165 effort=0 velocity=0 -> lower=-5 upper=3.867 effort=0 velocity=0; origin xyz=-0.020448 0.11835 0.0083512 rpy=-1.5672 1.5708 0 -> xyz=-0.022225 0.17977 0.0074 rpy=1.5708 0 -3.1416
- joint joint_5: origin xyz=-0.0010724 -2.0879E-05 0.08245 rpy=1.5708 -0.0035837 -1.5708 -> xyz=0 0.00165 0.07925 rpy=1.5708 0 -3.1416
- joint joint_6: limit lower=-1.565 upper=1.565 effort=0 velocity=0 -> lower=-1.6 upper=1.6 effort=0 velocity=0; origin xyz=-0.014463 0.080052 0.001425 rpy=1.5744 -1.5708 0 -> xyz=-0.01475 0.08 0.001425 rpy=1.5708 0 0

Commit message: Runtime dependencies and Simulation Support (#11)
* fixed outdated message references. added udev rules for arm

* added wait time for startup procedure on low-power embedded systems

* gazebo simulation re-resolved

* filled in erroneous effort and velocity limits in urdf

* adds simulation flag

* fixes namespace incompatibility between gazebo and moveits expected controller space. incorrect inertial and mass values corrected for link_4 and link_3

* new PID for trajectory. better controller plugin management

* reorganizing launch files

File: svenzva_description/robots/svenzva_arm.urdf (robot description, URDF)
Before this commit: robot revel, 10 links, 9 joints
Links:
- link link_3: mass 0.227860881806706 -> 0.285860881806706
- link link_4: mass 0.174540765744632 -> 0.236769
Joints:
- joint finger_joint_1: limit lower=0 upper=0.05 effort=0 velocity=0 -> lower=0 upper=0.05 effort=100 velocity=10
- joint finger_joint_2: limit lower=-0.05 upper=0 effort=0 velocity=0 -> lower=-0.05 upper=0 effort=100 velocity=10
- joint joint_1: limit lower=-3.14 upper=3.14 effort=0 velocity=0 -> lower=-3.14 upper=3.14 effort=100 velocity=10
- joint joint_2: limit lower=-2 upper=2 effort=0 velocity=0 -> lower=-2 upper=2 effort=100 velocity=10
- joint joint_3: limit lower=-2 upper=2 effort=0 velocity=0 -> lower=-2 upper=2 effort=100 velocity=10
- joint joint_4: limit lower=-5 upper=3.867 effort=0 velocity=0 -> lower=-3 upper=3 effort=10 velocity=1
- joint joint_5: limit lower=-1.7 upper=1.7 effort=0 velocity=0 -> lower=-1.7 upper=1.7 effort=100 velocity=10
- joint joint_6: limit lower=-1.6 upper=1.6 effort=0 velocity=0 -> lower=-1.6 upper=1.6 effort=100 velocity=10

Commit message: changed inertial parameters

File: svenzva_description/robots/svenzva_arm.urdf (robot description, URDF)
Before this commit: robot revel, 10 links, 9 joints
Links:
- link link_1: mass 0.295038974095265 -> 0.095038974095265

Commit message: Driver, URDF, Utilities bug fixes and updates (#14)
* forced joint1 to be 0 in model. adds new time derivative torque boost for joint 1

* fixes issue in detecting when to end trajectory action server. fixes missing reference. KT server now uses a special loader that preserves yaml order.

* adds python dependency for yaml ordered loading

* changed inertial parameters

* sped up arm parameters. added gripper open, close scripts. correctly setup utils package for library importing

* added medium speed controller parmas. fixed bug in joy node

* fixed issue in kt gui where gripper actions were not written

* added param

* added and cleaned up interaction files. added example file for how to use KT file as library

* added new urdf

* changed gripper limits in accordance with offset change

* changed gear ratios

* limit changes

* fixed button issue with custom controller. updated gear ratio and error message for cartesian control

* added optional collision checking for cartesian movements

* mode RRTConnect default planner

* changed method of collision detection

* added buffer zone above ground plane

* changed time dertivative, limited reliance on moveit being brough up

* increased opening torque

* changed delay for gripper

* now makes hard assumption that fingers are initialized correctly

* makes joint movement intuitive for linear motions

* added parameter for enabling velocity checking, added end effector link, tested new ways to find singularities

* added wall collisions

* switched joysticks on controller

* added new smoothing heuristic

* new heuristic. fixed ros parameter resolution

* updates urdf. launched cartesian controller conditionally

* adds updated urdf.

* adds standalone kinematics solver and replaces numerical solver

* fixes console gui hanging after kt playback

* urdf update

* updates to kinematics and joint limits

* gear ratio changes

* updated spring force eq

* updates references to mesh

* added dae textures

File: svenzva_description/robots/svenzva_arm.urdf (robot description, URDF)
Before this commit: robot revel, 10 links, 9 joints
Links:
- added link ee_link
- link base_link: mass 0.722020764728074 -> 0.673945611735726; geometry collision mesh filename=package://svenzva_description/meshes/base_link.STL; visual mesh filename=package://svenzva_description/textures/base_link.dae
- link link_1: mass 0.295038974095265 -> 0.386092665970672; geometry collision mesh filename=package://svenzva_description/meshes/link_1.STL; visual mesh filename=package://svenzva_description/textures/link_1.dae
- link link_2: mass 0.350557648873674 -> 0.63194; geometry collision mesh filename=package://svenzva_description/meshes/link_2.STL; visual mesh filename=package://svenzva_description/textures/link_2.dae
- link link_3: mass 0.285860881806706 -> 0.37014; geometry collision mesh filename=package://svenzva_description/meshes/link_3.STL; visual mesh filename=package://svenzva_description/textures/link_3.dae
- link link_4: mass 0.236769 -> 0.208577727676899; geometry collision mesh filename=package://svenzva_description/meshes/link_4.STL; visual mesh filename=package://svenzva_description/textures/link_4.dae
- link link_5: mass 0.133021865517638 -> 0.198143515414093; geometry collision mesh filename=package://svenzva_description/meshes/link_5.STL; visual mesh filename=package://svenzva_description/textures/link_5.dae
- link link_6: mass 0.243320868551208 -> 0.217466355310719; geometry collision mesh filename=package://svenzva_description/meshes/link_6.STL; visual mesh filename=package://svenzva_description/textures/link_6.dae
Joints:
- added joint ee_joint: type fixed, parent link_6, child ee_link, origin xyz=0 0 -0.05 rpy=3.14159 0 0
- joint finger_joint_1: axis -1 0 0 -> 0 -1 0
- joint finger_joint_2: axis -1 0 0 -> 0 -1 0
- joint joint_1: limit lower=-3.14 upper=3.14 effort=100 velocity=10 -> lower=-3.14 upper=3.14 effort=10 velocity=1; origin xyz=0 0 0.0762 rpy=0 0 0 -> xyz=0 0 0.064752 rpy=0 0 0
- joint joint_2: limit lower=-2 upper=2 effort=100 velocity=10 -> lower=-2.0 upper=2.0 effort=10 velocity=1; origin xyz=-0.007325 0 0.10542 rpy=1.5708 0 -1.5708 -> xyz=0.00039444 -0.0064686 0.11076 rpy=1.5708 0 0
- joint joint_3: axis 0 0 -1 -> 0 0 1; limit lower=-2 upper=2 effort=100 velocity=10 -> lower=-2.5 upper=2.5 effort=10 velocity=1; origin xyz=0 0.2277 0.00635 rpy=3.1416 0 3.1416 -> xyz=0 0.26625 0.014294 rpy=0 0 0
- joint joint_4: axis 0 0 1 -> 0 0 -1; limit lower=-3 upper=3 effort=10 velocity=1 -> lower=-4.5 upper=2.5 effort=10 velocity=1; origin xyz=-0.022225 0.17977 0.0074 rpy=1.5708 0 -3.1416 -> xyz=0 0.13713 -0.015019 rpy=-1.5708 0 0
- joint joint_5: axis 0 0 -1 -> 0 1 0; limit lower=-1.7 upper=1.7 effort=100 velocity=10 -> lower=-1.8 upper=1.8 effort=10 velocity=1; origin xyz=0 0.00165 0.07925 rpy=1.5708 0 -3.1416 -> xyz=0 -0.0040438 0.086925 rpy=0 0 0
- joint joint_6: limit lower=-1.6 upper=1.6 effort=100 velocity=10 -> lower=0.0 upper=5.85 effort=10 velocity=1; origin xyz=-0.01475 0.08 0.001425 rpy=1.5708 0 0 -> xyz=0 -0.019119 0.082 rpy=3.1416 0 3.1416

Commit message: New Joystick  (#15)
* added full support for 3axis joystick

* renamed 2axis controller to 6axis for accuracy

* resolves issue with nondeterministic crashes on launch

* adds missing runtime dependencies, eliminates old debug output, updates udev rules

* modified joint limit for shorter wrist cable

* adds greater flexibility for joint 6

* fixes inversed joystick movements

* updates example collisions for moveit

File: svenzva_description/robots/svenzva_arm.urdf (robot description, URDF)
Before this commit: robot revel, 11 links, 10 joints
Joints:
- joint joint_6: limit lower=0.0 upper=5.85 effort=10 velocity=1 -> lower=0.2 upper=5.5 effort=10 velocity=1

Commit message: makes joint limits more conservative for exibit. adds timer for gripper motor for safety. shortens distance fingers open.

File: svenzva_description/robots/svenzva_arm.urdf (robot description, URDF)
Before this commit: robot revel, 11 links, 10 joints
Joints:
- joint joint_1: limit lower=-3.14 upper=3.14 effort=10 velocity=1 -> lower=-1.570795 upper=1.570795 effort=10 velocity=1
- joint joint_2: limit lower=-2.0 upper=2.0 effort=10 velocity=1 -> lower=-1.7 upper=1.7 effort=10 velocity=1
- joint joint_3: limit lower=-2.5 upper=2.5 effort=10 velocity=1 -> lower=-2.5 upper=1.0 effort=10 velocity=1

Commit message: added and switched to joint control velocity control and added joint limits that make motion smoother and appropriate

File: svenzva_description/robots/svenzva_arm.urdf (robot description, URDF)
Before this commit: robot revel, 11 links, 10 joints
Joints:
- joint joint_4: limit lower=-4.5 upper=2.5 effort=10 velocity=1 -> lower=-4.5 upper=-1.4 effort=10 velocity=1

Commit message: changes to joint limits for resting, init position

File: svenzva_description/robots/svenzva_arm.urdf (robot description, URDF)
Before this commit: robot revel, 11 links, 10 joints
Joints:
- joint joint_4: limit lower=-4.5 upper=-1.4 effort=10 velocity=1 -> lower=-3.5 upper=1.0 effort=10 velocity=1

Commit message: Arm motor generalization (#17)
* adds parameters for customized builds that may not have a gripper.

* imposes safe joint limits for spring-assembly on joint 2

* modifications to allow joint trajectory controller to handle less than 7 joints

* general clean up

* dynamics module can now handle robots with non-default number of joints

File: svenzva_description/robots/svenzva_arm.urdf (robot description, URDF)
Before this commit: robot revel, 11 links, 10 joints
Joints:
- joint joint_2: limit lower=-2.0 upper=2.0 effort=10 velocity=1 -> lower=-1.5 upper=1.5 effort=10 velocity=1

Commit message: Add modularity to the Revel description files via Xacro (#20)
* adds base xacro file

* cleans up finger mesh files, fixes bug with finger distance in model

* additional changes to fingers to standarize their origin. adds additional finger type

* additional offset changes to fingers for greater accuracy and modularity. adds two accessories

* cleanup to make set default arm parameters. Adds in moveit config

* adds new finger type, and ability to change fingers in xacro

File: svenzva_description/robots/svenzva_arm.urdf (robot description, URDF)
Before this commit: robot revel, 11 links, 10 joints
Links:
- removed link finger_joint_2
- added link finger_link_2, mass 0.0220307791071739; collision mesh filename=package://svenzva_description/meshes/accessories/finger_sta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; visual mesh filename=package://svenzva_description/meshes/accessories/finger_sta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
- link finger_link_1: geometry collision mesh filename=package://svenzva_description/meshes/accessories/finger_sta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; visual mesh filename=package://svenzva_description/meshes/accessories/finger_sta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
Joints:
- joint finger_joint_1: origin xyz=0 0 -0.052509 rpy=-3.1416 -1.8964E-18 3.1416 -> xyz=0 0 -0.052002 rpy=-3.1416 0 3.1416
- joint finger_joint_2: axis 0 -1 0 -> 0 1 0; child finger_joint_2 -> finger_link_2; limit lower=-0.05 upper=0 effort=100 velocity=10 -> lower=0 upper=0.05 effort=100 velocity=10; origin xyz=0 0 -0.052509 rpy=-3.1416 -1.8964E-18 3.1416 -> xyz=0 0 -0.052002 rpy=-3.1416 0 3.1416
